Commit message: 5DOF URDF, ikin with level tip

File: src/basic134/urdf/example.urdf (robot description, URDF)
Before this commit: robot example, 9 links, 8 joints
Links:
- added link fingermotor; visual mesh filename=package://basic134/meshes/X5.stl scale=0.001 0.001 0.001
- added link hand; visual mesh filename=package://basic134/meshes/link_short.STL scale=0.001 0.001 0.001
- added link lbracket2; visual mesh filename=package://operation/meshes/lbracket2.STL scale=0.001 0.001 0.001
- added link wristmotor; visual mesh filename=package://basic134/meshes/X5.stl scale=0.001 0.001 0.001
- link lowerarm: geometry visual mesh filename=package://basic134/meshes/link.STL scale=0.001 0.001 0.001
Joints:
- added joint finger: type continuous, parent fingermotor, child tip, origin xyz=0 0 .0311 rpy=0 0 0, axis 0 0 1
- added joint hand: type fixed, parent hand, child lbracket2, origin xyz=0 0.15266 0 rpy=0 0 0
- added joint lbracket2: type fixed, parent lbracket2, child fingermotor, origin xyz=.045 0 -0.0525 rpy=-1.5708 0 -1.5708
- added joint wrist: type continuous, parent wristmotor, child hand, origin xyz=0 0 .0311 rpy=0 0 0, axis 0 0 1
- joint lowerarm: child tip -> wristmotor; origin xyz=0.315 0 0.003175 rpy=0 0 0 -> xyz=0 0.30095 0 rpy=0 3.1415 1.5708
- joint upperarm: origin xyz=-0.3 0 0 rpy=0 3.1415 0 -> xyz=0 0.3 0 rpy=0 3.1415 -1.5708
