Commit message: final commit

File: src/install/basic134/share/basic134/urdf/example.urdf (robot description, URDF)
Before this commit: robot example, 13 links, 12 joints
Links:
- added link magnet; visual cylinder length=0.021 radius=0.01
Joints:
- added joint magnet: type fixed, parent magnet, child tip, origin xyz=0 0 0.025 rpy=0 0 0
- joint finger: child tip -> magnet

File: src/install/operation/share/operation/urdf/example.urdf (robot description, URDF)
Before this commit: robot example, 13 links, 12 joints
Links:
- removed link basemotor
- removed link elbowmotor
- removed link fingermotor
- removed link hand
- removed link lbracket
- removed link lbracket2
- removed link lowerarm
- removed link shouldermotor
- removed link upperarm
- removed link wristmotor
- added link basecylinder; visual cylinder length=0.0127 radius=0.2286
- added link motor0; visual sphere radius=0.000001
- added link motor1; visual sphere radius=0.025
- added link motor1link; visual cylinder length=0.0902 radius=0.0254
- added link motor2; visual cylinder length=0.1 radius=0.02
- added link motor2link; visual cylinder length=0.396 radius=0.016
- added link motor3; visual cylinder length=0.1 radius=0.02
- added link motor3link; visual cylinder length=0.396 radius=0.016
- added link motor4; visual cylinder length=0.1 radius=0.02
- added link motor4link; visual cylinder length=0.1535 radius=0.016
- added link tiplink; visual cylinder length=0.1275 radius=0.016
- link baseplate: geometry visual box size=0.1778 0.1778 0.05
Joints:
- removed joint base
- removed joint elbow
- removed joint finger
- removed joint hand
- removed joint lbracket
- removed joint lbracket2
- removed joint lowerarm
- removed joint shoulder
- removed joint upperarm
- removed joint wrist
- added joint basecylinder: type fixed, parent basecylinder, child motor1link, origin xyz=0 0 0.0127 rpy=0 0 0
- added joint motor1link: type fixed, parent motor1link, child motor1, origin xyz=0.0225 0.017 0.0902 rpy=0 0 0
- added joint motor2link: type fixed, parent motor2link, child motor2, origin xyz=0.0574 0.396 0.0 rpy=0 0 0
- added joint motor3link: type fixed, parent motor3link, child motor3, origin xyz=-0.0574 0.396 0.0 rpy=0 0 0
- added joint motor4link: type fixed, parent motor4link, child motor4, origin xyz=0 0.1535 0.0574 rpy=0 0 0
- added joint theta0: type continuous, parent motor0, child basecylinder, origin xyz=0 0 0 rpy=0 0 0, axis 0 0 1
- added joint theta1: type continuous, parent motor1, child motor2link, origin xyz=0 0 0 rpy=0 0 0, axis 1 0 0
- added joint theta2: type continuous, parent motor2, child motor3link, origin xyz=0 0 0 rpy=0 0 0, axis 1 0 0
- added joint theta3: type continuous, parent motor3, child motor4link, origin xyz=0 0 0 rpy=0 0 0, axis 1 0 0
- added joint theta4: type continuous, parent motor4, child tiplink, origin xyz=0 0 0 rpy=0 0 0, axis 0 0 1
- added joint tiplink: type fixed, parent tiplink, child tip, origin xyz=0 0.1275 0 rpy=0 0 0
- joint baseplate: child basemotor -> motor0; origin xyz=0.08 0 0.012 rpy=0 0 0 -> xyz=0 0 0 rpy=0 0 0
